File: MainBoard/PoolTable.brd (EAGLE design)
At the start: 185.4 x 178.3 mm, 54 parts, among them IC6 LM317MBSTT3, J1 2X6 FEMALE, J2 2X6 FEMALE, J3 FEMALE 2x3, J4 FEMALE 2x3, M0 MOLEX-ULTRAFIT-1X03-VERT, M1 MOLEX-ULTRAFIT-1X03VERT, M2 MOLEX-ULTRAFIT-1X03VERT, M3 MOLEX-ULTRAFIT-1X03VERT, M4 MOLEX-ULTRAFIT-1X03VERT, M5 MOLEX-ULTRAFIT-1X03VERT, M6 MOLEX-ULTRAFIT-1X03VERT, M7 MOLEX-ULTRAFIT-1X03VERT, M8 MOLEX-ULTRAFIT-1X03-VERT, Q1 60V/32A/35mΩ, Q2 60V/32A/35mΩ, Q3 60V/32A/35mΩ, Q4 60V/32A/35mΩ, Q5 60V/32A/35mΩ, Q6 60V/32A/35mΩ, Q7 60V/32A/35mΩ, Q8 60V/32A/35mΩ, Q9 60V/32A/35mΩ, U1 TMP102, U2 TMP102, U3 TMP102, U4 TMP102

Commit message: Auto stash before merge of "master" and "origin/master"
Routing:
- net R1: track 0.00 -> 71.3 mm
- net R2: track 0.00 -> 61.9 mm
- net G1: track 0.00 -> 61.8 mm
- net G2: track 0.00 -> 51.7 mm
- net B1: track 2.54 -> 51.5 mm
- net R3: track 0.00 -> 48.4 mm
- net B2: track 0.00 -> 40.3 mm
- net G3: track 0.00 -> 37.5 mm
- net B3: track 0.00 -> 26.1 mm
Other:
- board text added: "5V"
- board text added: "5v"
- board text added: "GND"
- board text added: "MISO"
- board text added: "MOSI"
- board text added: "SCL"
- board text added: "SCLK"
- board text added: "SDA"
- board text added: "SS"
Changed lines of the file:
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@@
 <text x="145.669" y="164.465" size="2.54" layer="25" rot="R180">S3</text>
 <text x="134.239" y="164.465" size="2.54" layer="25" rot="R180">S4</text>
+<text x="8.89" y="147.32" size="0.635" layer="21" rot="R180" align="center">SCL</text>
+<text x="11.43" y="147.32" size="0.635" layer="21" rot="R180" align="center">5v</text>
+<text x="3.81" y="147.32" size="0.635" layer="21" rot="R180" align="center">GND</text>
+<text x="6.35" y="147.32" size="0.635" layer="21" rot="R180" align="center">SDA</text>
+<text x="3.81" y="121.92" size="0.635" layer="21" align="center">5V</text>
+<text x="13.97" y="121.92" size="0.635" layer="21" align="center">5V</text>
+<text x="19.05" y="121.92" size="0.635" layer="21" align="center">GND</text>
+<text x="8.89" y="121.92" size="0.635" layer="21" align="center">GND</text>
+<text x="6.35" y="121.92" size="0.635" layer="21" align="center">SS</text>
+<text x="16.51" y="121.92" size="0.635" layer="21" align="center">SS</text>
+<text x="3.81" y="129.54" size="0.635" layer="21" align="center">MISO</text>
+<text x="6.35" y="128.905" size="0.635" layer="21" align="center">MOSI</text>
+<text x="8.89" y="129.54" size="0.635" layer="21" align="center">SCLK</text>
+<text x="13.97" y="129.54" size="0.635" layer="21" align="center">MISO</text>
+<text x="16.51" y="128.905" size="0.635" layer="21" align="center">MOSI</text>
+<text x="19.05" y="129.54" size="0.635" layer="21" align="center">SCLK</text>
 </plain>
 <attributes>
@@
 </element>
 <element name="J3" library="SparkFun-Connectors" package="2X3" value="FEMALE 2x3" x="3.81" y="124.46" smashed="yes">
-<attribute name="NAME" x="2.54" y="128.524" size="0.6096" layer="25" font="vector" ratio="20"/>
 <attribute name="PROD_ID" value="CONN-11566" x="3.81" y="124.46" size="1.778" layer="27" display="off"/>
-<attribute name="VALUE" x="2.54" y="122.047" size="0.6096" layer="27" font="vector" ratio="20"/>
 </element>
 <element name="J4" library="SparkFun-Connectors" package="2X3" value="FEMALE 2x3" x="13.97" y="124.46" smashed="yes">
-<attribute name="NAME" x="12.7" y="128.524" size="0.6096" layer="25" font="vector" ratio="20"/>
 <attribute name="PROD_ID" value="CONN-11566" x="13.97" y="124.46" size="1.778" layer="27" display="off"/>
-<attribute name="VALUE" x="12.7" y="122.047" size="0.6096" layer="27" font="vector" ratio="20"/>
 </element>
 </elements>
@@
 <contactref element="Q1" pad="1"/>
 <contactref element="PWM1" pad="PWM0"/>
-<wire x1="136.271" y1="156.337" x2="92.71" y2="130.81" width="0" layer="19" extent="1-1"/>
+<wire x1="128.27" y1="128.27" x2="95.25" y2="128.27" width="0.254" layer="16"/>
+<wire x1="92.71" y1="130.81" x2="95.25" y2="128.27" width="0.254" layer="16"/>
+<wire x1="139.7" y1="139.7" x2="139.7" y2="153.67" width="0.254" layer="16"/>
+<wire x1="139.7" y1="153.67" x2="137.033" y2="156.337" width="0.254" layer="16"/>
+<wire x1="137.033" y1="156.337" x2="136.271" y2="156.337" width="0.254" layer="16"/>
+<wire x1="128.27" y1="128.27" x2="139.7" y2="139.7" width="0.254" layer="16"/>
 </signal>
 <signal name="G1">
 <contactref element="Q2" pad="1"/>
 <contactref element="PWM1" pad="PWM1"/>
-<wire x1="136.271" y1="148.59" x2="92.71" y2="133.35" width="0" layer="19" extent="1-1"/>
+<wire x1="128.27" y1="129.54" x2="96.52" y2="129.54" width="0.254" layer="16"/>
+<wire x1="92.71" y1="133.35" x2="96.52" y2="129.54" width="0.254" layer="16"/>
+<wire x1="128.27" y1="129.54" x2="138.43" y2="139.7" width="0.254" layer="16"/>
+<wire x1="138.43" y1="139.7" x2="138.43" y2="147.32" width="0.254" layer="16"/>
+<wire x1="138.43" y1="147.32" x2="137.16" y2="148.59" width="0.254" layer="16"/>
+<wire x1="137.16" y1="148.59" x2="136.271" y2="148.59" width="0.254" layer="16"/>
 </signal>
 <signal name="B1">
 <contactref element="Q3" pad="1"/>
 <contactref element="PWM1" pad="PWM2"/>
-<wire x1="136.271" y1="141.351" x2="138.811" y2="141.351" width="0.635" layer="1"/>
-<wire x1="138.811" y1="141.351" x2="92.71" y2="135.89" width="0" layer="19" extent="1-1"/>
+<wire x1="128.27" y1="130.81" x2="97.79" y2="130.81" width="0.254" layer="16"/>
+<wire x1="92.71" y1="135.89" x2="97.79" y2="130.81" width="0.254" layer="16"/>
+<wire x1="128.27" y1="130.81" x2="136.271" y2="138.811" width="0.254" layer="16"/>
+<wire x1="136.271" y1="138.811" x2="136.271" y2="141.351" width="0.254" layer="16"/>
 </signal>
 <signal name="N$1">
@@
 <contactref element="Q4" pad="1"/>
 <contactref element="PWM1" pad="PWM3"/>
-<wire x1="123.571" y1="156.337" x2="92.71" y2="138.43" width="0" layer="19" extent="1-1"/>
+<wire x1="92.71" y1="138.43" x2="99.06" y2="132.08" width="0.254" layer="16"/>
+<wire x1="99.06" y1="132.08" x2="121.92" y2="132.08" width="0.254" layer="16"/>
+<wire x1="121.92" y1="132.08" x2="128.27" y2="138.43" width="0.254" layer="16"/>
+<wire x1="128.27" y1="138.43" x2="128.27" y2="153.67" width="0.254" layer="16"/>
+<wire x1="125.603" y1="156.337" x2="123.571" y2="156.337" width="0.254" layer="16"/>
+<wire x1="128.27" y1="153.67" x2="125.603" y2="156.337" width="0.254" layer="16"/>
 </signal>
 <signal name="G2">
 <contactref element="Q5" pad="1"/>
 <contactref element="PWM1" pad="PWM4"/>
-<wire x1="123.571" y1="148.59" x2="92.71" y2="140.97" width="0" layer="19" extent="1-1"/>
+<wire x1="92.71" y1="140.97" x2="100.33" y2="133.35" width="0.254" layer="16"/>
+<wire x1="100.33" y1="133.35" x2="121.92" y2="133.35" width="0.254" layer="16"/>
+<wire x1="121.92" y1="133.35" x2="127" y2="138.43" width="0.254" layer="16"/>
+<wire x1="127" y1="138.43" x2="127" y2="146.05" width="0.254" layer="16"/>
+<wire x1="127" y1="146.05" x2="124.46" y2="148.59" width="0.254" layer="16"/>
+<wire x1="124.46" y1="148.59" x2="123.571" y2="148.59" width="0.254" layer="16"/>
 </signal>
 <signal name="B2">
 <contactref element="Q6" pad="1"/>
 <contactref element="PWM1" pad="PWM5"/>
-<wire x1="123.571" y1="141.351" x2="92.71" y2="143.51" width="0" layer="19" extent="1-1"/>
+<wire x1="92.71" y1="143.51" x2="101.6" y2="134.62" width="0.254" layer="16"/>
+<wire x1="101.6" y1="134.62" x2="121.92" y2="134.62" width="0.254" layer="16"/>
+<wire x1="121.92" y1="134.62" x2="123.571" y2="136.271" width="0.254" layer="16"/>
+<wire x1="123.571" y1="136.271" x2="123.571" y2="141.351" width="0.254" layer="16"/>
 </signal>
 <signal name="R3">
 <contactref element="Q7" pad="1"/>
 <contactref element="PWM1" pad="PWM6"/>
-<wire x1="110.871" y1="156.337" x2="92.71" y2="146.05" width="0" layer="19" extent="1-1"/>
+<wire x1="92.71" y1="146.05" x2="102.87" y2="135.89" width="0.254" layer="16"/>
+<wire x1="102.87" y1="135.89" x2="110.49" y2="135.89" width="0.254" layer="16"/>
+<wire x1="110.49" y1="135.89" x2="115.57" y2="140.97" width="0.254" layer="16"/>
+<wire x1="115.57" y1="140.97" x2="115.57" y2="154.94" width="0.254" layer="16"/>
+<wire x1="115.57" y1="154.94" x2="114.173" y2="156.337" width="0.254" layer="16"/>
+<wire x1="114.173" y1="156.337" x2="110.871" y2="156.337" width="0.254" layer="16"/>
 </signal>
 <signal name="G3">
 <contactref element="Q8" pad="1"/>
 <contactref element="PWM1" pad="PWM7"/>
-<wire x1="110.871" y1="148.59" x2="92.71" y2="148.59" width="0" layer="19" extent="1-1"/>
+<wire x1="92.71" y1="148.59" x2="104.14" y2="137.16" width="0.254" layer="16"/>
+<wire x1="104.14" y1="137.16" x2="110.49" y2="137.16" width="0.254" layer="16"/>
+<wire x1="110.49" y1="137.16" x2="114.3" y2="140.97" width="0.254" layer="16"/>
+<wire x1="114.3" y1="140.97" x2="114.3" y2="146.05" width="0.254" layer="16"/>
+<wire x1="114.3" y1="146.05" x2="111.76" y2="148.59" width="0.254" layer="16"/>
+<wire x1="111.76" y1="148.59" x2="110.871" y2="148.59" width="0.254" layer="16"/>
 </signal>
 <signal name="B3">
 <contactref element="Q9" pad="1"/>
 <contactref element="PWM1" pad="PWM8"/>
-<wire x1="92.71" y1="151.13" x2="110.871" y2="141.351" width="0" layer="19" extent="1-1"/>
+<wire x1="92.71" y1="151.13" x2="105.41" y2="138.43" width="0.254" layer="16"/>
+<wire x1="110.871" y1="138.811" x2="110.871" y2="141.351" width="0.254" layer="16"/>
+<wire x1="105.41" y1="138.43" x2="110.49" y2="138.43" width="0.254" layer="16"/>
+<wire x1="110.49" y1="138.43" x2="110.871" y2="138.811" width="0.254" layer="16"/>
 </signal>
 <signal name="N$4">

Commit message: pool table final
Parts:
- added U$1: (no value), SparkFun-Aesthetics:OSHW-LOGO-L
Routing:
- net N$5: track 0.00 -> 222.5 mm, vias 0 -> 3
- net N$4: track 0.00 -> 220.0 mm, vias 0 -> 3
- net N$18: track 0.00 -> 143.8 mm
- net N$19: track 0.00 -> 136.0 mm, vias 0 -> 1
- net N$17: track 0.00 -> 129.6 mm
- net SS1: track 0.00 -> 106.6 mm, vias 0 -> 3
- net SS2: track 0.00 -> 99.8 mm, vias 0 -> 1
- net CPU0_SDA0: track 326.9 -> 419.5 mm
- net 5V: track 530.8 -> 598.7 mm
- net CPU0_SCL0: track 388.2 -> 442.8 mm
- net GND: track 0.00 -> 7.24 mm, vias 2 -> 4
- net 3.3V: track 449.6 -> 451.9 mm
- net 1.8V: track 337.3 -> 338.9 mm
Other:
- board text added: "PoolTable Backplane Created by DART 2019 Released under the GPLv3"
