File: Modules/CPU.brd (EAGLE design)
At the start: 132.1 x 55.5 mm, 89 parts, among them IC4 93LC66SM, IC5 MIC2026-1YM, J1 USB_A_SMT_FEMALE, J2 USB_A_SMT_FEMALE, J4 SD_CARD_SOCKET, Q1 DMG1012T-7, Q2 DMG1012T-7, Q3 DMG1012T-7, U5 LAN9512-JZX, U6 FSUSB42UMX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

Commit message: Updated CPU Module and removed components from Main Board
Parts:
- moved C22 292.6 mm to (196.7, 115.6), flipped to the bottom, turned to 90 degrees
- moved C21 290.2 mm to (198.1, 115.6), flipped to the bottom, turned to 90 degrees
- moved C20 283.6 mm to (195.3, 115.6), flipped to the bottom, turned to 90 degrees
- moved C19 278.4 mm to (193.9, 115.6), flipped to the bottom, turned to 90 degrees
- moved FB2 273.0 mm to (188.2, 115.4), flipped to the bottom, turned to 90 degrees
- moved C34 236.2 mm to (179.1, 102.9), flipped to the bottom, turned to 90 degrees
- moved C33 231.0 mm to (177.7, 102.9), flipped to the bottom, turned to 90 degrees
- moved C31 226.2 mm to (180.3, 108.0), flipped to the bottom, turned to 90 degrees
- moved C32 225.8 mm to (176.3, 102.9), flipped to the bottom, turned to 90 degrees
- moved C30 221.0 mm to (178.9, 108.0), flipped to the bottom, turned to 90 degrees
- moved C25 215.9 mm to (192.5, 115.6), flipped to the bottom, turned to 90 degrees
- moved C29 215.8 mm to (177.5, 108.0), flipped to the bottom, turned to 90 degrees
- moved C24 210.7 mm to (191.1, 115.6), flipped to the bottom, turned to 90 degrees
- moved C28 210.6 mm to (176.1, 108.0), flipped to the bottom, turned to 90 degrees
- moved C23 205.5 mm to (189.7, 115.6), flipped to the bottom, turned to 90 degrees
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